File: vein-finder-organic/ee/kicad/vein_finder.kicad_sch (KiCad schematic)
At the start: 67 parts, among them J1 USB-C power-only, Q1 AO3400A, Q2 AO3400A, SW1 B3F-1020, U1 ATtiny1614, U2 BQ21040DBVR, U3 TPS61169

Commit message: Vein finder (organic): fixes from a full self-review
Firmware (host tests and AVR build pass; not yet on hardware):
- clear the stale sleep request after waking, so a press is not lost and the
  part does not go straight back to power-down
- sleep only if the button and USB are still idle, read with interrupts off,
  so an edge taken by the pin ISR just before sleep cannot be lost
- wait for WDT SYNCBUSY before each CTRLA write
- an open NTC (ADC >= 1000) counts as over-temperature: LEDs off (it read as
  0 C and silently disabled the 41 C limit); new tests
- timing on the real 15.625 ms tick (auto-off exactly 180 s, hold 594 ms)

Scripts and outputs:
- placement reads courtyards with the S-expression parser (the regex leaked
  silk lines); placement unchanged, about 27x faster with the vectorised room
  check; room cache rebuilt when the layout is newer
- silk tidy restores a text it cannot place; finisher: no duplicate widths,
  final connectivity re-check, rip-ups counted for lost GND pads
- Edge.Cuts DXF without the plated pin holes; schematic regenerated with the
  re-checked sourcing text (40 nets, 0 mismatches)
- iec62471.py reads the LED power from optics.json; stale comments, figure
  labels and doc numbers corrected

Co-Authored-By: Claude Opus 5.5 <noreply@anthropic.com>
Claude-Session: https://claude.ai/code/session_01VQzXs58X1YYUn6JuF7hh2E
Parts:
- BT1: Verified A: $10.81 @1, 1,637 in stock (snippet; other snapshots 93-1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 -> A (re-checked 2026-10-12): $10.81 @1, 1,637 in stock (digik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
- C1: Verified A: $0.0064 @50+ (MOQ 50), 6.3 M in stock (snippet) -> A (re-checked 2026-10-12): $0.0064-0.0225 @50+ (MOQ 50; cac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
- C3: Verified A: $0.015 @100+, 7.8-13.3 M in stock (snippets) -> A (re-checked 2026-10-12): $0.0085-0.016 @100+ (cached page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
- C5: Verified A: $0.0221 @10+, 573,070 in stock (snippet) -> A (re-checked 2026-10-12): $0.022-0.0492 @10+ (cached pages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
- C7: Verified A: $0.0191 @20+, 484,120 in stock (snippet; 'not recommende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 -> A (re-checked 2026-10-12): $0.1764 @5+ on the product page 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
- D1: Verified A: 47,700-145,260 in stock (snippets); qty-10 price NV ($0.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 -> A (re-checked 2026-10-12): $0.055-0.061 @10+ (MOQ 10; highe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
- D14: Verified A: $0.0221 @20+ (MOQ 20), 54-56 k in stock (snippets); 591 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 -> A (re-checked 2026-10-12): $0.0215-0.0248 @20+ (MOQ 20; hig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
- D2: Verified A: $0.67 @1, $0.462 @10, ~20,945 in stock (snippets); 660 n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 -> A (re-checked 2026-10-12): $0.69-0.70 @1, $0.48-0.54 @10 (t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
- D8: Verified A: $0.51 @1, $0.354 @10; stock 870-10,870 (snippets disagre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 -> A (re-checked 2026-10-12): $0.48 @1, $0.326 @10, 16,312 in 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
- H1: Verified A: 47,494 in stock (snippet); price NV; 5.84 mm posts -> A (re-checked 2026-10-12): $1.23 @1, $1.04 @10, 46-48 k in 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
- J1: Verified A: $0.61 @1, 11,429 in stock (digikey.com snippet); Mouser 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 -> A (re-checked 2026-10-12): $0.61 @1, 11,429 in stock (digik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
- L1: Verified A: $0.0594 @10+, 1,459 in stock (snippet); Isat 1.30 A, DCR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 -> A (re-checked 2026-10-12): $0.0594 @10+, 1,459 in stock (on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
- Q1: Verified A: $0.076-0.083 @5+, 100 k-1.14 M in stock (snippets); 30 V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 -> A (re-checked 2026-10-12): $0.0735-0.0898 @5+ (cached pages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
- R1: Verified A: $0.0012-0.0016 @100+, 2.4-4.0 M in stock (snippets) -> A (re-checked 2026-10-12): $0.0015-0.0026 @100+ (cached pag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
- R13: Verified A: $0.0011 @100+, ~9.9 M in stock (snippet) -> A (re-checked 2026-10-12): $0.0037-0.0058 @100+ (cached pag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
- R3: Verified A: $0.0013-0.0015 @100+, 0.47-3.7 M in stock (snippets) -> A (re-checked 2026-10-12): $0.0018-0.0041 @100+ (cached pag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
- R4: Verified A: $0.0014 @100+, 9.03 M in stock (snippet) -> A (re-checked 2026-10-12): $0.0014-0.0034 @100+ (cached pag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
- R5: Verified A: about $0.001 @100+, 1.5-2.3 M in stock (snippets) -> A (re-checked 2026-10-12): $0.0014-0.0047 @100+ (cached pag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
- R9: Verified A: $0.0035 @100+, 2,300-8,600 in stock (snippets) -> A (re-checked 2026-10-12): $0.0054 @100+, 2,300 in stock
- RT1: Verified A: ~$0.03 @10, 510-722 k in stock (snippets) -> A (re-checked 2026-10-12): $0.0295-0.0467 @10+ (cached page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
- SW1: Verified A: from $0.071, 1,940 in stock (snippet); 5.0 mm, 0.98 N, 0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 -> A (re-checked 2026-10-12): $0.1523 @5+ (MOQ 5; the earlier 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
- U1: Verified A: $0.90 @1, 33,040 in stock (digikey.com snippet) -> A (re-checked 2026-10-12): $0.90 @1, 33,040 in stock (digik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
- U2: Verified A: $0.3148-0.3303 @5+ (MOQ 5), 960-2,860 in stock (snippets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 -> A (re-checked 2026-10-12): $0.2542-0.3303 @5+ (MOQ 5; cache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
- U3: Verified A: 8,475-8,970 in stock, $0.16-0.33 @5+ (MOQ 5; two snapsho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 -> A (re-checked 2026-10-12): $0.1606-0.3268 @5+ (MOQ 5; cache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
